File: feeder/pcb/mobo/mobo.kicad_pcb (KiCad board)
At the start: 2 copper layers, 200 x 100 mm, 86 parts, among them J1 SWD_10, J2 FTDI_HEADER, J3 PLATED_PADS, M1 PEEL_MOTOR, M2 DRIVE_MOTOR, SW1 RESET, SW2 BUTTON_1, SW3 BUTTON_2, SW4 BOOT, U1 QRE1113, U2 STM32F103C8Tx, U3 TCS40DPR, U4 AP1117-33, U5 MCP16301, U6 DRV8833PWP, U7 MAX3078E, Y1 8MHz

Commit message: Lock labels
Parts:
- added ?: , buzzard_labels, F.Cu at (190.0, 57.6)
- added ?: , buzzard_labels, F.Cu at (187.2, 60.1)
- added G***: LOGO, index:logo, F.Cu at (178.3, 58.8)
